Commit message: Created Core URDF

File: src/my_robot/description/robot_core.xacro (robot description, xacro)
@@ -1,3 +1,112 @@
 <?xml version="1.0"?>
-<robot xmlns:xacro="http://www.ros.org/wiki/xacro" >
+<robot xmlns:xacro="http://www.ros.org/wiki/xacro">
+     <xacro:include filename="inertial_macros.xacro"/>
+  <!-- MATERIALS -->
+  <material name="white">
+    <color rgba="1 1 1 1"/>
+  </material>
+  <material name="orange">
+    <color rgba="1 0.3 0.1 1"/>
+  </material>
+  <material name="blue">
+    <color rgba="0.2 0.2 1 1"/>
+  </material>
+  <material name="black">
+    <color rgba="0 0 0 1"/>
+  </material>
+  <!-- BASE LINK -->
+  <link name="base_link">
+  </link>
+  <!-- CHASSIS LINK -->
+  <joint name="chassis_joint" type="fixed">
+    <parent link="base_link"/>
+    <child link="chassis_link"/>
+    <origin xyz="-0.1 0 0"/>
+  </joint>
+  <link name="chassis_link">
+    <visual>
+      <origin xyz="0.15 0 0.075"/>
+      <geometry>
+        <box size="0.3 0.3 0.15"/>
+      </geometry>
+      <material name="white"/>
+    </visual>
+    <collision>
+      <origin xyz="0.15 0 0.075"/>
+      <geometry>
+        <box size="0.3 0.3 0.15"/>
+      </geometry>
+    </collision>
+    <xacro:inertial_box mass="0.5" x="0.3" y="0.3" z="0.15">
+    <origin xyz="0.15 0 0.075" rpy="0 0 0"/>
+    </xacro:inertial_box>
+  </link>
+  <!-- LEFT WHEEL -->
+  <joint name="left_wheel_joint" type="continuous">
+    <parent link="base_link"/>
+    <child link="left_wheel_link"/>
+    <origin xyz="0 0.175 0" rpy="-${pi/2} 0.0 0.0"/>
+    <axis xyz="0 0 1"/>
+  </joint>
+  <link name="left_wheel_link">
+    <visual>
+      <geometry>
+        <cylinder radius="0.05" length="0.04"/>
+      </geometry>
+      <material name="blue"/>
+    </visual>
+    <collision>
+      <geometry>
+        <cylinder radius="0.05" length="0.04"/>
+      </geometry>
+    </collision>
+     <xacro:inertial_cylinder mass="0.1" length="0.04" radius="0.05">
+    <origin xyz="0 0 0" rpy="0 0 0"/>
+    </xacro:inertial_cylinder>
+  </link>
+  <!-- RIGHT WHEEL -->
+  <joint name="right_wheel_joint" type="continuous">
+    <parent link="base_link"/>
+    <child link="right_wheel_link"/>
+    <origin xyz="0 -0.175 0" rpy="-${pi/2} 0.0 0.0"/>
+    <axis xyz="0 0 -1"/>
+  </joint>
+  <link name="right_wheel_link">
+    <visual>
+      <geometry>
+        <cylinder radius="0.05" length="0.04"/>
+      </geometry>
+      <material name="blue"/>
+    </visual>
+    <collision>
+      <geometry>
+        <cylinder radius="0.05" length="0.04"/>
+      </geometry>
+    </collision>
+     <xacro:inertial_cylinder mass="0.1" length="0.04" radius="0.05">
+    <origin xyz="0 0 0" rpy="0 0 0"/>
+    </xacro:inertial_cylinder>
+  </link>
+  <!-- CASTER WHEEL LINK -->
+  <joint name="caster_wheel_joint" type="fixed">
+    <parent link="chassis_link"/>
+    <child link="caster_wheel_link"/>
+    <origin xyz="0.24 0 0"/>
+  </joint>
+  <link name="caster_wheel_link">
+    <visual>
+      <geometry>
+        <sphere radius="0.05"/>
+      </geometry>
+      <material name="black"/>
+    </visual>
+    <collision>
+      <geometry>
+        <sphere radius="0.05"/>
+      </geometry>
+    </collision>
+     <xacro:inertial_sphere mass="0.1" radius="0.05">
+    <origin xyz="0 0 0" rpy="0 0 0"/>
+    </xacro:inertial_sphere>
+  </link>
 </robot>

Commit message: Add launch_sim file and update robot core xacro

File: src/my_robot/description/robot_core.xacro (robot description, xacro)
@@ -42,4 +42,7 @@
     </xacro:inertial_box>
   </link>
+  <gazebo reference="chassis_link">
+  <material>Gazebo/White</material>
+  </gazebo>
   <!-- LEFT WHEEL -->
   <joint name="left_wheel_joint" type="continuous">
@@ -65,4 +68,7 @@
     </xacro:inertial_cylinder>
   </link>
+  <gazebo reference="left_wheel_link">
+  <material>Gazebo/Blue</material>
+  </gazebo>
   <!-- RIGHT WHEEL -->
   <joint name="right_wheel_joint" type="continuous">
@@ -88,4 +94,7 @@
     </xacro:inertial_cylinder>
   </link>
+  <gazebo reference="right_wheel_link">
+  <material>Gazebo/Blue</material>
+  </gazebo>
   <!-- CASTER WHEEL LINK -->
   <joint name="caster_wheel_joint" type="fixed">
@@ -110,3 +119,6 @@
     </xacro:inertial_sphere>
   </link>
+  <gazebo reference="caster_wheel_link">
+  <material>Gazebo/Black</material>
+  </gazebo>
 </robot>

Commit message: feat(simulation): setup mobile robot in Gazebo with obstacle world

File: src/my_robot/description/robot_core.xacro (robot description, xacro)
@@ -75,5 +75,5 @@
     <parent link="base_link"/>
     <child link="right_wheel_link"/>
-    <origin xyz="0 -0.175 0" rpy="-${pi/2} 0.0 0.0"/>
+    <origin xyz="0 -0.175 0" rpy="${pi/2} 0.0 0.0"/>
     <axis xyz="0 0 -1"/>
   </joint>
@@ -121,4 +121,6 @@
   <gazebo reference="caster_wheel_link">
   <material>Gazebo/Black</material>
+  <mu1 value="0.001"/>
+    <mu2 value="0.001"/>
   </gazebo>
 </robot>
